File: level-shifter.sch (KiCad schematic (older format))
At the start: 13 parts

Commit message: change 3.3 to VCC to satisfy rules check
Parts:
- gave numbers to parts that had none: 7
Connections:
- net labels added: VCC
- net labels removed: +3.3V
Changed lines of the file:
@@
-EESchema Schematic File Version 2  date Sat 21 Jan 2012 01:36:10 PM CET
+EESchema Schematic File Version 2  date Sat 21 Jan 2012 01:41:20 PM CET
 LIBS:power
 LIBS:device
@@
 Comment4 ""
 $EndDescr
+$Comp
+L VCC #PWR01
+U 1 1 4F1AB249
+P 3300 750
+F 0 "#PWR01" H 3300 850 30  0001 C CNN
+F 1 "VCC" H 3300 850 30  0000 C CNN
+	1    3300 750
+	1    0    0    -1
+$EndComp
 Wire Wire Line
 	4200 6800 4200 7000
@@
 Connection ~ 3300 6400
 $Comp
-L GND #PWR01
+L GND #PWR02
 U 1 1 4F1AB0CB
 P 4200 7000
-F 0 "#PWR01" H 4200 7000 30  0001 C CNN
+F 0 "#PWR02" H 4200 7000 30  0001 C CNN
 F 1 "GND" H 4200 6930 30  0001 C CNN
 	1    4200 7000
@@
 $EndComp
 $Comp
-L C C?
+L C C2
 U 1 1 4F1AB05F
 P 4200 6600
-F 0 "C?" H 4250 6700 50  0000 L CNN
+F 0 "C2" H 4250 6700 50  0000 L CNN
 F 1 "1uF" H 4250 6500 50  0000 L CNN
 	1    4200 6600
@@
 $EndComp
 $Comp
-L C C?
+L C C1
 U 1 1 4F1AB050
 P 4250 1800
-F 0 "C?" H 4300 1900 50  0000 L CNN
+F 0 "C1" H 4300 1900 50  0000 L CNN
 F 1 "1uF" H 4300 1700 50  0000 L CNN
 	1    4250 1800
@@
 P 4150 850
 AR Path="/4F1AAF5E" Ref="#FLG?"  Part="1"
-AR Path="/4F1AAF64" Ref="#FLG02"  Part="1"
-F 0 "#FLG02" H 4150 1120 30  0001 C CNN
+AR Path="/4F1AAF64" Ref="#FLG03"  Part="1"
+F 0 "#FLG03" H 4150 1120 30  0001 C CNN
 F 1 "PWR_FLAG" H 4150 1080 30  0000 C CNN
 	1    4150 850
@@
 $EndComp
 $Comp
-L PWR_FLAG #FLG03
+L PWR_FLAG #FLG04
 U 1 1 4F1AAF5E
 P 5000 850
-F 0 "#FLG03" H 5000 1120 30  0001 C CNN
+F 0 "#FLG04" H 5000 1120 30  0001 C CNN
 F 1 "PWR_FLAG" H 5000 1080 30  0000 C CNN
 	1    5000 850
@@
 $EndComp
 $Comp
-L GND #PWR04
+L GND #PWR05
 U 1 1 4F1AAF38
 P 4700 1400
-F 0 "#PWR04" H 4700 1400 30  0001 C CNN
+F 0 "#PWR05" H 4700 1400 30  0001 C CNN
 F 1 "GND" H 4700 1330 30  0001 C CNN
 	1    4700 1400
@@
 $EndComp
 $Comp
-L CONN_2 P?
+L CONN_2 P1
 U 1 1 4F1AAEFA
 P 4600 700
-F 0 "P?" V 4550 700 40  0000 C CNN
+F 0 "P1" V 4550 700 40  0000 C CNN
 F 1 "CONN_2" V 4650 700 40  0000 C CNN
 	1    4600 700
 	0    -1   -1   0
-$EndComp
-$Comp
-L +3.3V #PWR05
-U 1 1 4F1AAE56
-P 3300 750
-F 0 "#PWR05" H 3300 710 30  0001 C CNN
-F 1 "+3.3V" H 3300 860 30  0000 C CNN
-	1    3300 750
-	1    0    0    -1
 $EndComp
 $Comp
@@
 P 4250 3750
 AR Path="/4F1AAB5B" Ref="P?"  Part="1"
-AR Path="/4F1AAB70" Ref="P?"  Part="1"
-F 0 "P?" V 4200 3750 60  0000 C CNN
+AR Path="/4F1AAB70" Ref="P3"  Part="1"
+F 0 "P3" V 4200 3750 60  0000 C CNN
 F 1 "CONN_8" V 4300 3750 60  0000 C CNN
 	1    4250 3750
@@
 $EndComp
 $Comp
-L CONN_8 P?
+L CONN_8 P2
 U 1 1 4F1AAB5B
 P 900 3750
-F 0 "P?" V 850 3750 60  0000 C CNN
+F 0 "P2" V 850 3750 60  0000 C CNN
 F 1 "CONN_8" V 950 3750 60  0000 C CNN
 	1    900  3750
@@
 $Comp
 L 74LS126 U?
-U 1 1 4F1AAAE4
+U 4 1 4F1AAAE4
 P 2450 6100
 AR Path="/4F1AAABA" Ref="U?"  Part="1"
-AR Path="/4F1AAAE4" Ref="U?"  Part="1"
-F 0 "U?" H 2550 6300 60  0000 C CNN
+AR Path="/4F1AAAE4" Ref="U2"  Part="4"
+F 0 "U2" H 2550 6300 60  0000 C CNN
 F 1 "74LS126" H 2700 5950 60  0000 C CNN
-	1    2450 6100
-	1    0    0    -1
-$EndComp
-$Comp
-L 74LS126 U?
-U 1 1 4F1AAAE2
+	4    2450 6100
+	1    0    0    -1
+$EndComp
+$Comp
+L 74LS126 U?
+U 3 1 4F1AAAE2
 P 2450 5450
 AR Path="/4F1AAABA" Ref="U?"  Part="1"
-AR Path="/4F1AAAE2" Ref="U?"  Part="1"
-F 0 "U?" H 2550 5650 60  0000 C CNN
+AR Path="/4F1AAAE2" Ref="U2"  Part="3"
+F 0 "U2" H 2550 5650 60  0000 C CNN
 F 1 "74LS126" H 2700 5300 60  0000 C CNN
-	1    2450 5450
-	1    0    0    -1
-$EndComp
-$Comp
-L 74LS126 U?
-U 1 1 4F1AAAE0
+	3    2450 5450
+	1    0    0    -1
+$EndComp
+$Comp
+L 74LS126 U?
+U 2 1 4F1AAAE0
 P 2450 4800
 AR Path="/4F1AAABA" Ref="U?"  Part="1"
-AR Path="/4F1AAAE0" Ref="U?"  Part="1"
-F 0 "U?" H 2550 5000 60  0000 C CNN
+AR Path="/4F1AAAE0" Ref="U2"  Part="2"
+F 0 "U2" H 2550 5000 60  0000 C CNN
 F 1 "74LS126" H 2700 4650 60  0000 C CNN
-	1    2450 4800
+	2    2450 4800
 	1    0    0    -1
 $EndComp
@@
 P 2450 4150
 AR Path="/4F1AAABA" Ref="U?"  Part="1"
-AR Path="/4F1AAADF" Ref="U?"  Part="1"
-F 0 "U?" H 2550 4350 60  0000 C CNN
+AR Path="/4F1AAADF" Ref="U2"  Part="1"
+F 0 "U2" H 2550 4350 60  0000 C CNN
 F 1 "74LS126" H 2700 4000 60  0000 C CNN
 	1    2450 4150
@@
 $Comp
 L 74LS126 U?
-U 1 1 4F1AAAD9
+U 4 1 4F1AAAD9
 P 2450 3250
 AR Path="/4F1AAABA" Ref="U?"  Part="1"
-AR Path="/4F1AAAD9" Ref="U?"  Part="1"
-F 0 "U?" H 2550 3450 60  0000 C CNN
+AR Path="/4F1AAAD9" Ref="U1"  Part="4"
+F 0 "U1" H 2550 3450 60  0000 C CNN
 F 1 "74LS126" H 2700 3100 60  0000 C CNN
-	1    2450 3250
-	1    0    0    -1
-$EndComp
-$Comp
-L 74LS126 U?
-U 1 1 4F1AAAD4
+	4    2450 3250
+	1    0    0    -1
+$EndComp
+$Comp
+L 74LS126 U?
+U 3 1 4F1AAAD4
 P 2450 2550
 AR Path="/4F1AAABA" Ref="U?"  Part="1"
-AR Path="/4F1AAAD4" Ref="U?"  Part="1"
-F 0 "U?" H 2550 2750 60  0000 C CNN
+AR Path="/4F1AAAD4" Ref="U1"  Part="3"
+F 0 "U1" H 2550 2750 60  0000 C CNN
 F 1 "74LS126" H 2700 2400 60  0000 C CNN
-	1    2450 2550
-	1    0    0    -1
-$EndComp
-$Comp
-L 74LS126 U?
-U 1 1 4F1AAACE
+	3    2450 2550
+	1    0    0    -1
+$EndComp
+$Comp
+L 74LS126 U?
+U 2 1 4F1AAACE
 P 2450 1850
 AR Path="/4F1AAABA" Ref="U?"  Part="1"
-AR Path="/4F1AAACE" Ref="U?"  Part="1"
-F 0 "U?" H 2550 2050 60  0000 C CNN
+AR Path="/4F1AAACE" Ref="U1"  Part="2"
+F 0 "U1" H 2550 2050 60  0000 C CNN
 F 1 "74LS126" H 2700 1700 60  0000 C CNN
-	1    2450 1850
-	1    0    0    -1
-$EndComp
-$Comp
-L 74LS126 U?
+	2    2450 1850
+	1    0    0    -1
+$EndComp
+$Comp
+L 74LS126 U1
 U 1 1 4F1AAABA
 P 2450 1200
-F 0 "U?" H 2550 1400 60  0000 C CNN
+F 0 "U1" H 2550 1400 60  0000 C CNN
 F 1 "74LS126" H 2700 1050 60  0000 C CNN
 	1    2450 1200
